Commit message: fix: detect legacy gazebo/franka import new one

File: gazebo-11/assets/robots/franka_panda/panda_description/urdf/panda.urdf (robot description, URDF)
Before this commit: robot panda, 12 links, 11 joints
Links:
- added link panda_grasptarget, mass 0.0
- link panda_hand: mass None -> .81; geometry collision mesh filename=package://meshes/collision/hand.obj; visual mesh filename=package://meshes/visual/hand.obj
- link panda_leftfinger: mass None -> 0.1; geometry collision mesh filename=package://meshes/collision/finger.obj; visual mesh filename=package://meshes/visual/finger.obj
- link panda_link0: mass None -> 2.9; geometry collision mesh filename=package://meshes/collision/link0.obj; visual mesh filename=package://meshes/collision/link0.obj
- link panda_link1: mass None -> 2.7; geometry collision mesh filename=package://meshes/collision/link1.obj; visual mesh filename=package://meshes/visual/link1.obj
- link panda_link2: mass None -> 2.73; geometry collision mesh filename=package://meshes/collision/link2.obj; visual mesh filename=package://meshes/visual/link2.obj
- link panda_link3: mass None -> 2.04; geometry collision mesh filename=package://meshes/collision/link3.obj; visual mesh filename=package://meshes/visual/link3.obj
- link panda_link4: mass None -> 2.08; geometry collision mesh filename=package://meshes/collision/link4.obj; visual mesh filename=package://meshes/visual/link4.obj
- link panda_link5: mass None -> 3; geometry collision mesh filename=package://meshes/collision/link5.obj; visual mesh filename=package://meshes/visual/link5.obj
- link panda_link6: mass None -> 1.3; geometry collision mesh filename=package://meshes/collision/link6.obj; visual mesh filename=package://meshes/visual/link6.obj
- link panda_link7: mass None -> .2; geometry collision mesh filename=package://meshes/collision/link7.obj; visual mesh filename=package://meshes/collision/link7.obj
- link panda_link8: mass None -> 0.0
- link panda_rightfinger: mass None -> 0.1; geometry collision mesh filename=package://meshes/collision/finger.obj; visual mesh filename=package://meshes/visual/finger.obj
Joints:
- added joint panda_grasptarget_hand: type fixed, parent panda_hand, child panda_grasptarget, origin xyz=0 0 0.105 rpy=0 0 0
- joint panda_joint1: limit lower=-2.9671 upper=2.9671 effort=87 velocity=2.3925 -> lower=-2.9671 upper=2.9671 effort=87 velocity=2.1750
- joint panda_joint2: limit lower=-1.8326 upper=1.8326 effort=87 velocity=2.3925 -> lower=-1.8326 upper=1.8326 effort=87 velocity=2.1750
- joint panda_joint3: limit lower=-2.9671 upper=2.9671 effort=87 velocity=2.3925 -> lower=-2.9671 upper=2.9671 effort=87 velocity=2.1750
- joint panda_joint4: limit lower=-3.1416 upper=0.0873 effort=87 velocity=2.3925 -> lower=-3.1416 upper=0.0 effort=87 velocity=2.1750
- joint panda_joint5: limit lower=-2.9671 upper=2.9671 effort=12 velocity=2.8710 -> lower=-2.9671 upper=2.9671 effort=12 velocity=2.6100
- joint panda_joint6: limit lower=-0.0873 upper=3.8223 effort=12 velocity=2.8710 -> lower=-0.0873 upper=3.8223 effort=12 velocity=2.6100
- joint panda_joint7: limit lower=-2.9671 upper=2.9671 effort=12 velocity=2.8710 -> lower=-2.9671 upper=2.9671 effort=12 velocity=2.6100
